File: board/nrfsensornode.sch (EAGLE design)
At the start: 16 parts, among them IC1 LM1117MPX-3.3, IC2 DS1820

Commit message: Updates
Parts:
- removed JP4: (no value), pinhead:PINHD-2X15
- removed VCC: (no value), adafruit:PINHD-1X15-CB
- added 1W, A0, A1, A2, A3, A4, A5, A6, A7, D10, D2, D3, D4, D6, D9: (no value), adafruit:PINHD-1X3
- added DHT**: 22-23-2041, con-molex:22-23-2041
- added R2: 4.7k, adafruit:R-US_M1206
- IC2: value DS1820 -> DS18b20
- R1: device adafruit:R-US_0204/7 -> adafruit:R-US_M1206
- renumbered JP1 to POWER, JP3 to NRF24L01, PAD1 to MISO, PAD2 to SCK, PAD3 to RESET, PAD4 to 5V, PAD5 to MOSI, PAD6 to GND
Connections:
- new net IC1COOL: IC1.NC
- net A0: now also A0.1; no longer JP4.1
- net A1: now also A1.1; no longer JP4.3
- net A2: now also A2.1; no longer JP4.5
- net A3: now also A3.1; no longer JP4.7
- net A4: now also A4.1; no longer JP4.9
- net A5: now also A5.1; no longer JP4.11
- net A6: now also A6.1; no longer JP4.13
- net A7: now also A7.1; no longer JP4.15
- net D10: now also D10.1; no longer JP4.29
- net D2: now also D2.1; no longer JP4.17
- net D3: now also D3.1, DHT**-2.S, R2.2; no longer JP4.19
- net D4: now also D4.1; no longer JP4.21
- net D5: now also 1W.1; no longer JP4.23
- net D6: now also D6.1; no longer JP4.25
- net D9: now also D9.1; no longer JP4.27
- net GND: now also 1W.2, A0.2, A1.2, A2.2, A3.2, A4.2, A5.2, A6.2, A7.2, D10.2, D2.2, D3.2, D4.2, D6.2, D9.2, DHT**-4.S; no longer JP4.10, JP4.12, JP4.14, JP4.16, JP4.18, JP4.2, JP4.20, JP4.22, JP4.24, JP4.26, JP4.28, JP4.30, JP4.4, JP4.6, JP4.8
- net RAW: now also 1W.3, A0.3, A1.3, A2.3, A3.3, A4.3, A5.3, A6.3, A7.3, D10.3, D2.3, D3.3, D4.3, D6.3, D9.3, DHT**-1.S, R2.1; no longer VCC.1, VCC.10, VCC.11, VCC.12, VCC.13, VCC.14, VCC.15, VCC.2, VCC.3, VCC.4, VCC.5, VCC.6, VCC.7, VCC.8, VCC.9
Other:
- moved on the sheet: R1

Commit message: Various changes
Parts:
- added R3: 10k, adafruit:R-US_M1206
- C1: value 10uf -> 22uf
Connections:
- net GND: now also R3.2
- net MISO: now also R3.1
Changed lines of the file:
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@@
 <part name="GND1" library="supply1" deviceset="GND" device=""/>
 <part name="IC1" library="v-reg-lm1117" deviceset="LM1117?*" device="MPX" technology="-3.3" value=""/>
-<part name="C1" library="adafruit" deviceset="CPOL-US" device="E2-4" value="10uf"/>
+<part name="C1" library="adafruit" deviceset="CPOL-US" device="E2-4" value="22uf"/>
 <part name="U$1" library="zarya" deviceset="ARDMINIPRO" device=""/>
 <part name="+3V1" library="supply1" deviceset="+3V3" device=""/>
@@
 <part name="D10" library="adafruit" deviceset="PINHD-1X3" device=""/>
 <part name="1W" library="adafruit" deviceset="PINHD-1X3" device=""/>
+<part name="R3" library="adafruit" deviceset="R-US_" device="M1206" value="10k"/>
 </parts>
 <sheets>
@@
 <instance part="D10" gate="A" x="-147.32" y="86.36"/>
 <instance part="1W" gate="A" x="-129.54" y="86.36"/>
+<instance part="R3" gate="G$1" x="12.7" y="43.18"/>
 </instances>
 <busses>
@@
 <pinref part="IC1" gate="G$1" pin="GND"/>
 <wire x1="33.02" y1="81.28" x2="33.02" y2="66.04" width="0.1524" layer="91"/>
-<wire x1="33.02" y1="66.04" x2="45.72" y2="66.04" width="0.1524" layer="91"/>
+<wire x1="33.02" y1="66.04" x2="38.1" y2="66.04" width="0.1524" layer="91"/>
 <pinref part="C1" gate="G$1" pin="-"/>
+<wire x1="38.1" y1="66.04" x2="45.72" y2="66.04" width="0.1524" layer="91"/>
 <wire x1="45.72" y1="73.66" x2="45.72" y2="66.04" width="0.1524" layer="91"/>
 <wire x1="0" y1="66.04" x2="20.32" y2="66.04" width="0.1524" layer="91"/>
@@
 <wire x1="20.32" y1="73.66" x2="20.32" y2="66.04" width="0.1524" layer="91"/>
 <label x="-2.54" y="58.42" size="1.27" layer="95" rot="R180" xref="yes"/>
+<wire x1="38.1" y1="66.04" x2="38.1" y2="43.18" width="0.1524" layer="91"/>
+<pinref part="R3" gate="G$1" pin="2"/>
+<wire x1="38.1" y1="43.18" x2="17.78" y2="43.18" width="0.1524" layer="91"/>
+<junction x="38.1" y="66.04"/>
 </segment>
 <segment>
@@
 <segment>
 <pinref part="NRF24L01" gate="A" pin="7"/>
-<wire x1="7.62" y1="50.8" x2="-2.54" y2="50.8" width="0.1524" layer="91"/>
+<wire x1="7.62" y1="50.8" x2="0" y2="50.8" width="0.1524" layer="91"/>
 <label x="-2.54" y="50.8" size="1.27" layer="95" rot="R180" xref="yes"/>
-</segment>
-<segment>
+<junction x="0" y="50.8"/>
+<wire x1="0" y1="50.8" x2="-2.54" y2="50.8" width="0.1524" layer="91"/>
+<wire x1="0" y1="50.8" x2="0" y2="43.18" width="0.1524" layer="91"/>
+<pinref part="R3" gate="G$1" pin="1"/>
+<wire x1="0" y1="43.18" x2="7.62" y2="43.18" width="0.1524" layer="91"/>
+</segment>
+<segment>

Commit message: updated libs updated board
Parts:
- added POWERSELECT: (no value), SparkFun-Connectors:M03X2POGO_PINS
Connections:
- removed net +5V: 5V.P, U$1.VCC
- removed net IC1COOL: IC1.NC
- new net A_RAW: POWERSELECT.1, U$1.RAW
- new net A_VCC: 5V.P, POWERSELECT.5, U$1.VCC
- new net NRF_VCC: NRF24L01.2, POWERSELECT.4
- net +3V3: now also IC1.NC, POWERSELECT.6; no longer NRF24L01.2
- net RAW: now also POWERSELECT.2, POWERSELECT.3; no longer U$1.RAW
Changed lines of the file:
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@@
 <part name="R1" library="adafruit" deviceset="R-US_" device="M1206" value="4.7k"/>
 <part name="C2" library="adafruit" deviceset="CPOL-US" device="E2-4" value="10uf"/>
-<part name="+3V2" library="supply1" deviceset="+3V3" device=""/>
 <part name="IC2" library="DS1820" deviceset="DS1820" device="" value="DS18b20"/>
 <part name="GND2" library="supply1" deviceset="GND" device=""/>
@@
 <part name="1W" library="adafruit" deviceset="PINHD-1X3" device=""/>
 <part name="R3" library="adafruit" deviceset="R-US_" device="M1206" value="10k"/>
+<part name="POWERSELECT" library="SparkFun-Connectors" deviceset="M03X2" device="POGO_PINS"/>
+<part name="+3V3" library="supply1" deviceset="+3V3" device=""/>
 </parts>
 <sheets>
@@
 <instance part="R1" gate="G$1" x="-127" y="38.1"/>
 <instance part="C2" gate="G$1" x="20.32" y="78.74"/>
-<instance part="+3V2" gate="G$1" x="25.4" y="58.42" rot="R270"/>
 <instance part="IC2" gate="G$1" x="-119.38" y="27.94"/>
 <instance part="GND2" gate="1" x="-119.38" y="15.24"/>
@@
 <instance part="1W" gate="A" x="-129.54" y="86.36"/>
 <instance part="R3" gate="G$1" x="12.7" y="43.18"/>
+<instance part="POWERSELECT" gate="G$1" x="-53.34" y="104.14"/>
+<instance part="+3V3" gate="G$1" x="-30.48" y="101.6" smashed="yes" rot="R270">
+<attribute name="VALUE" x="-30.48" y="101.6" size="1.778" layer="96"/>
+</instance>
 </instances>
 <busses>
@@
 </segment>
 </net>
-<net name="+5V" class="0">
-<segment>
-<pinref part="U$1" gate="G$1" pin="VCC"/>
-<wire x1="-71.12" y1="76.2" x2="-71.12" y2="86.36" width="0.1524" layer="91"/>
-<label x="-71.12" y="86.36" size="1.27" layer="95" rot="MR90" xref="yes"/>
-</segment>
-<segment>
-<pinref part="5V" gate="G$1" pin="P"/>
-<wire x1="-134.62" y1="119.38" x2="-129.54" y2="119.38" width="0.1524" layer="91"/>
-<label x="-129.54" y="119.38" size="1.016" layer="95" xref="yes"/>
-</segment>
-</net>
 <net name="D10" class="0">
 <segment>
@@
 </net>
 <net name="RAW" class="0">
-<segment>
-<pinref part="U$1" gate="G$1" pin="RAW"/>
-<wire x1="-86.36" y1="76.2" x2="-86.36" y2="86.36" width="0.1524" layer="91"/>
-<label x="-86.36" y="86.36" size="1.27" layer="95" rot="MR90" xref="yes"/>
-</segment>
 <segment>
 <pinref part="POWER" gate="G$1" pin="1"/>
@@
 <label x="-154.94" y="83.82" size="1.27" layer="95" rot="MR0" xref="yes"/>
 </segment>
+<segment>
+<pinref part="POWERSELECT" gate="G$1" pin="3"/>
+<wire x1="-60.96" y1="104.14" x2="-68.58" y2="104.14" width="0.1524" layer="91"/>
+<label x="-68.58" y="104.14" size="1.27" layer="95" rot="R180" xref="yes"/>
+</segment>
+<segment>
+<pinref part="POWERSELECT" gate="G$1" pin="2"/>
+<wire x1="-45.72" y1="106.68" x2="-35.56" y2="106.68" width="0.1524" layer="91"/>
+<label x="-35.56" y="106.68" size="1.27" layer="95" xref="yes"/>
+</segment>
 </net>
 <net name="SCK" class="0">
@@
 </segment>
 <segment>
-<pinref part="NRF24L01" gate="A" pin="2"/>
-<wire x1="22.86" y1="58.42" x2="15.24" y2="58.42" width="0.1524" layer="91"/>
-<pinref part="+3V2" gate="G$1" pin="+3V3"/>
+<pinref part="POWERSELECT" gate="G$1" pin="6"/>
+<wire x1="-45.72" y1="101.6" x2="-33.02" y2="101.6" width="0.1524" layer="91"/>
+<pinref part="+3V3" gate="G$1" pin="+3V3"/>
+</segment>
+<segment>
+<pinref part="IC1" gate="G$1" pin="NC"/>
+<wire x1="35.56" y1="96.52" x2="35.56" y2="101.6" width="0.1524" layer="91"/>
 </segment>
 </net>
@@
 </segment>
 </net>
-<net name="IC1COOL" class="0">
-<segment>
-<pinref part="IC1" gate="G$1" pin="NC"/>
-<wire x1="35.56" y1="96.52" x2="35.56" y2="101.6" width="0.1524" layer="91"/>
-</segment>
-</net>
+<net name="NRF_VCC" class="0">
+<segment>
+<pinref part="POWERSELECT" gate="G$1" pin="4"/>
+<wire x1="-45.72" y1="104.14" x2="-40.64" y2="104.14" width="0.1524" layer="91"/>
+<label x="-40.64" y="104.14" size="1.27" layer="95" xref="yes"/>
+</segment>
+<segment>
+<pinref part="NRF24L01" gate="A" pin="2"/>
+<wire x1="22.86" y1="58.42" x2="15.24" y2="58.42" width="0.1524" layer="91"/>
+<label x="22.86" y="58.42" size="1.27" layer="95" xref="yes"/>
+</segment>
+</net>
+<net name="A_VCC" class="0">
+<segment>
+<pinref part="U$1" gate="G$1" pin="VCC"/>
+<wire x1="-71.12" y1="76.2" x2="-71.12" y2="86.36" width="0.1524" layer="91"/>
+<label x="-71.12" y="86.36" size="1.27" layer="95" rot="MR90" xref="yes"/>
+</segment>
+<segment>
+<pinref part="POWERSELECT" gate="G$1" pin="5"/>
+<wire x1="-60.96" y1="101.6" x2="-68.58" y2="101.6" width="0.1524" layer="91"/>
+<label x="-68.58" y="101.6" size="1.27" layer="95" rot="MR0" xref="yes"/>
+</segment>
+<segment>
+<pinref part="5V" gate="G$1" pin="P"/>
+<wire x1="-134.62" y1="119.38" x2="-129.54" y2="119.38" width="0.1524" layer="91"/>
+<label x="-129.54" y="119.38" size="1.016" layer="95" xref="yes"/>
+</segment>
+</net>
+<net name="A_RAW" class="0">
+<segment>
+<pinref part="U$1" gate="G$1" pin="RAW"/>
+<wire x1="-86.36" y1="76.2" x2="-86.36" y2="86.36" width="0.1524" layer="91"/>
+<label x="-86.36" y="86.36" size="1.27" layer="95" rot="MR90" xref="yes"/>
+</segment>
+<segment>
+<pinref part="POWERSELECT" gate="G$1" pin="1"/>
+<wire x1="-60.96" y1="106.68" x2="-68.58" y2="106.68" width="0.1524" layer="91"/>
+<label x="-68.58" y="106.68" size="1.27" layer="95" rot="R180" xref="yes"/>
+</segment>
+</net>

Commit message: Updates
Parts:
- added SHT1X: SHT1X, sht10_11_15:SHT1X
- D2, D3: device adafruit:PINHD-1X3 -> SparkFun-Connectors:M04LOCK
- renumbered RESET to RST
Connections:
- new net NRF_INT: D2.1, D3.1, NRF24L01.8
- net D2: now also D2.2; no longer D2.1
- net D3: now also D3.2, SHT1X.DATA; no longer D3.1
- net D4: now also SHT1X.SCK
- net GND: now also D2.3, D3.3, SHT1X.GND; no longer D2.2, D3.2
- net RAW: now also D2.4, D3.4, SHT1X.VDD; no longer D2.3, D3.3
Other:
- moved on the sheet: DHT**-1, DHT**-2, DHT**-3, DHT**-4, R2
